Commit message: still working...

File: mobile_robot_description/urdf/mobile_robot.urdf (robot description, URDF)
Before this commit: robot mobile_robot, 5 links, 4 joints
Links:
- link base_link: mass 2.0 -> 10.0
- link caster_wheel: mass 0.2 -> 1.0

Commit message: Simulation simple differential drive in Gazebo

File: mobile_robot_description/urdf/mobile_robot.urdf (robot description, URDF)
Before this commit: robot mobile_robot, 5 links, 4 joints
Links:
- link base_link: mass 10.0 -> 2.0
- link caster_wheel: mass 1.0 -> 0.5

Commit message: Add laser sensor

File: mobile_robot_description/urdf/mobile_robot.urdf (robot description, URDF)
Before this commit: robot mobile_robot, 5 links, 4 joints
Links:
- added link laser_link, mass 0.1; collision cylinder length=0.02 radius=0.02; visual cylinder length=0.02 radius=0.02
Joints:
- added joint laser_fixed_joint: type fixed, parent base_link, child laser_link, origin xyz=0.04 0 0.09 rpy=0 0 0

Commit message: Add xacro macro

File: mobile_robot_description/urdf/mobile_robot.urdf (robot description, URDF)
Before this commit: robot mobile_robot, 6 links, 5 joints
Links:
- removed link l_wheel
- removed link r_wheel
Joints:
- removed joint l_wheel_joint
- removed joint r_wheel_joint
