Commit message: Adjust link4_1 location

File: manipulator1_robot_description/urdf/robot.urdf.xacro (robot description, xacro)
@@ -57,5 +57,5 @@
         <origin xyz="0 0 0.1" rpy="0 0 0"/>
         <axis xyz="0 0 1"/>
-        <limit effort="1000" velocity="0.2" lower="${-pi}" upper="${pi}"/>
+        <limit effort="1000" velocity="1.0" lower="${-pi}" upper="${pi}"/>
     </joint>
     <transmission name="joint1_tran">
@@ -97,5 +97,5 @@
         <origin xyz="0 0.05 0.25" rpy="0 0 0"/>
         <axis xyz="0 1 0"/>
-        <limit effort="1000" velocity="0.2" lower="${-pi}" upper="${pi}"/>
+        <limit effort="1000" velocity="1.0" lower="${-pi}" upper="${pi}"/>
     </joint>
     <transmission name="joint2_tran">
@@ -137,5 +137,5 @@
         <origin xyz="0 0 0.4" rpy="0 0 0"/>
         <axis xyz="0 1 0"/>
-        <limit effort="1000" velocity="0.2" lower="${-pi}" upper="${pi}"/>
+        <limit effort="1000" velocity="1.0" lower="${-pi}" upper="${pi}"/>
     </joint>
     <transmission name="joint3_tran">
@@ -175,5 +175,5 @@
         <origin xyz="0 -0.05 0.15" rpy="0 0 0"/>
         <axis xyz="0 0 1"/>
-        <limit effort="1000" velocity="0.2" lower="${-pi}" upper="${pi}"/>
+        <limit effort="1000" velocity="1.0" lower="${-pi}" upper="${pi}"/>
     </joint>
     <transmission name="joint4_tran">
@@ -211,5 +211,5 @@
         <parent link="link4"/>
         <child link="link4_1"/>
-        <origin xyz="0 0.05 0.05" rpy="0 0 0"/>
+        <origin xyz="0 0.05 0.15" rpy="0 0 0"/>
     </joint>
     <link name="link5">
@@ -238,5 +238,5 @@
         <origin xyz="0 0 0.3" rpy="0 0 0"/>
         <axis xyz="0 1 0"/>
-        <limit effort="1000" velocity="0.2" lower="${-pi}" upper="${pi}"/>
+        <limit effort="1000" velocity="1.0" lower="${-pi}" upper="${pi}"/>
     </joint>
     <transmission name="joint5_tran">
@@ -276,5 +276,5 @@
         <origin xyz="0 -0.05 0.08" rpy="0 0 0"/>
         <axis xyz="0 0 1"/>
-        <limit effort="1000" velocity="0.2" lower="${-pi}" upper="${pi}"/>
+        <limit effort="1000" velocity="1.0" lower="${-pi}" upper="${pi}"/>
     </joint>
     <transmission name="joint6_tran">

Commit message: Add ik_tutorial package and adjust limit value of joints

File: manipulator1_robot_description/urdf/robot.urdf.xacro (robot description, xacro)
@@ -97,5 +97,5 @@
         <origin xyz="0 0.05 0.25" rpy="0 0 0"/>
         <axis xyz="0 1 0"/>
-        <limit effort="1000" velocity="1.0" lower="${-pi}" upper="${pi}"/>
+        <limit effort="1000" velocity="1.0" lower="-2.0" upper="2.0"/>
     </joint>
     <transmission name="joint2_tran">
@@ -137,5 +137,5 @@
         <origin xyz="0 0 0.4" rpy="0 0 0"/>
         <axis xyz="0 1 0"/>
-        <limit effort="1000" velocity="1.0" lower="${-pi}" upper="${pi}"/>
+        <limit effort="1000" velocity="1.0" lower="-2.0" upper="2.0"/>
     </joint>
     <transmission name="joint3_tran">
@@ -238,5 +238,5 @@
         <origin xyz="0 0 0.3" rpy="0 0 0"/>
         <axis xyz="0 1 0"/>
-        <limit effort="1000" velocity="1.0" lower="${-pi}" upper="${pi}"/>
+        <limit effort="1000" velocity="1.0" lower="-2.0" upper="2.0"/>
     </joint>
     <transmission name="joint5_tran">
